File: hardware/basicsensormodule.kicad_pcb (KiCad board)
At the start: 2 copper layers, 130.2 x 52.1 mm, 77 parts, among them J102 SENSOR, J401 USART, J601 RJ45, J602 RJ45, U201 MCP2551-I/SN, U202 MCP2515-xSO, U301 LM324, U401 ATMEGA328P-PU, U501 LM7805, Y201 16MHz, Y401 16MHz

Commit message: layout finalizado
Parts:
- removed C301, C302, C303, C304: 100n, Capacitor_SMD:C_0805_2012Metric_Pad1.15x1.40mm_HandSolder
- removed D101: LL4148, Diode_SMD:D_MiniMELF_Handsoldering
- removed D301: 4V7, Diode_SMD:D_MiniMELF_Handsoldering
- removed J102: SENSOR, TerminalBlock:TerminalBlock_bornier-4_P5.08mm
- removed JP101: jmp, Jumper:SolderJumper-3_P1.3mm_Open_RoundedPad1.0x1.5mm
- removed R301, R303, R304, R308, R309: 10k, Resistor_SMD:R_0805_2012Metric_Pad1.15x1.40mm_HandSolder
- removed R302: 100k, Resistor_SMD:R_0805_2012Metric_Pad1.15x1.40mm_HandSolder
- removed R305, R306, R307: 1k, Resistor_SMD:R_0805_2012Metric_Pad1.15x1.40mm_HandSolder
- removed TP301: op_a_in-, TestPoint:TestPoint_Pad_2.0x2.0mm
- removed TP302: op_a_out, TestPoint:TestPoint_Pad_2.0x2.0mm
- removed TP303: in-, TestPoint:TestPoint_Pad_2.0x2.0mm
- removed TP304: op_b_out, TestPoint:TestPoint_Pad_2.0x2.0mm
- removed TP305: op_b_in+, TestPoint:TestPoint_Pad_2.0x2.0mm
- removed TP306: in+, TestPoint:TestPoint_Pad_2.0x2.0mm
- removed TP307: op_a_in+, TestPoint:TestPoint_Pad_2.0x2.0mm
- removed U301: LM324, Package_SO:SOIC-14_3.9x8.7mm_P1.27mm
- added C102: 100nF, Capacitor_SMD:C_0805_2012Metric_Pad1.15x1.40mm_HandSolder, B.Cu at (237.5, 43.4)
- added C102: 100nF, Capacitor_SMD:C_0805_2012Metric_Pad1.15x1.40mm_HandSolder, B.Cu at (172.5, 43.4)
- added C102: 100nF, Capacitor_SMD:C_0805_2012Metric_Pad1.15x1.40mm_HandSolder, B.Cu at (107.5, 43.4)
- added C201: 100nF, Capacitor_SMD:C_0805_2012Metric_Pad1.15x1.40mm_HandSolder, B.Cu at (235.0, 94.0)
- added C201: 100nF, Capacitor_SMD:C_0805_2012Metric_Pad1.15x1.40mm_HandSolder, B.Cu at (170.0, 94.0)
- added C201: 100nF, Capacitor_SMD:C_0805_2012Metric_Pad1.15x1.40mm_HandSolder, B.Cu at (105.0, 94.0)
- added C202: 100nF, Capacitor_SMD:C_0805_2012Metric_Pad1.15x1.40mm_HandSolder, B.Cu at (242.6, 109.9)
- added C202: 100nF, Capacitor_SMD:C_0805_2012Metric_Pad1.15x1.40mm_HandSolder, B.Cu at (177.6, 109.9)
- added C202: 100nF, Capacitor_SMD:C_0805_2012Metric_Pad1.15x1.40mm_HandSolder, B.Cu at (112.6, 109.9)
- added C203: 22pF, Capacitor_SMD:C_0805_2012Metric_Pad1.15x1.40mm_HandSolder, B.Cu at (227.4, 100.1)
- added C203: 22pF, Capacitor_SMD:C_0805_2012Metric_Pad1.15x1.40mm_HandSolder, B.Cu at (162.4, 100.1)
- added C203: 22pF, Capacitor_SMD:C_0805_2012Metric_Pad1.15x1.40mm_HandSolder, B.Cu at (97.4, 100.1)
- added C204: 22pF, Capacitor_SMD:C_0805_2012Metric_Pad1.15x1.40mm_HandSolder, B.Cu at (229.5, 96.3)
- added C204: 22pF, Capacitor_SMD:C_0805_2012Metric_Pad1.15x1.40mm_HandSolder, B.Cu at (164.5, 96.3)
- added C204: 22pF, Capacitor_SMD:C_0805_2012Metric_Pad1.15x1.40mm_HandSolder, B.Cu at (99.5, 96.3)
- added C205: 100nF, Capacitor_SMD:C_0805_2012Metric_Pad1.15x1.40mm_HandSolder, B.Cu at (237.8, 119.8)
- added C205: 100nF, Capacitor_SMD:C_0805_2012Metric_Pad1.15x1.40mm_HandSolder, B.Cu at (172.8, 119.8)
- added C205: 100nF, Capacitor_SMD:C_0805_2012Metric_Pad1.15x1.40mm_HandSolder, B.Cu at (107.8, 119.8)
- added C401: 100nF, Capacitor_SMD:C_0805_2012Metric_Pad1.15x1.40mm_HandSolder, B.Cu at (246.1, 73.4)
- added C401: 100nF, Capacitor_SMD:C_0805_2012Metric_Pad1.15x1.40mm_HandSolder, B.Cu at (181.1, 73.4)
- added C401: 100nF, Capacitor_SMD:C_0805_2012Metric_Pad1.15x1.40mm_HandSolder, B.Cu at (116.1, 73.4)
- added C402: 100nF, Capacitor_SMD:C_0805_2012Metric_Pad1.15x1.40mm_HandSolder, B.Cu at (230.8, 68.3)
- added C402: 100nF, Capacitor_SMD:C_0805_2012Metric_Pad1.15x1.40mm_HandSolder, B.Cu at (165.8, 68.3)
- added C402: 100nF, Capacitor_SMD:C_0805_2012Metric_Pad1.15x1.40mm_HandSolder, B.Cu at (100.8, 68.3)
- added C403: 22pF, Capacitor_SMD:C_0805_2012Metric_Pad1.15x1.40mm_HandSolder, B.Cu at (228.3, 75.9)
- added C403: 22pF, Capacitor_SMD:C_0805_2012Metric_Pad1.15x1.40mm_HandSolder, B.Cu at (163.3, 75.9)
- added C403: 22pF, Capacitor_SMD:C_0805_2012Metric_Pad1.15x1.40mm_HandSolder, B.Cu at (98.3, 75.9)
- added C404: 22pF, Capacitor_SMD:C_0805_2012Metric_Pad1.15x1.40mm_HandSolder, B.Cu at (229.5, 71.5)
- added C404: 22pF, Capacitor_SMD:C_0805_2012Metric_Pad1.15x1.40mm_HandSolder, B.Cu at (164.5, 71.5)
- added C404: 22pF, Capacitor_SMD:C_0805_2012Metric_Pad1.15x1.40mm_HandSolder, B.Cu at (99.5, 71.5)
- added C405: 100nF, Capacitor_SMD:C_0805_2012Metric_Pad1.15x1.40mm_HandSolder, B.Cu at (229.5, 53.1)
- added C405: 100nF, Capacitor_SMD:C_0805_2012Metric_Pad1.15x1.40mm_HandSolder, B.Cu at (164.5, 53.1)
- added C405: 100nF, Capacitor_SMD:C_0805_2012Metric_Pad1.15x1.40mm_HandSolder, B.Cu at (99.5, 53.1)
- added C406: 100nF, Capacitor_SMD:C_0805_2012Metric_Pad1.15x1.40mm_HandSolder, B.Cu at (232.0, 48.1)
- added C406: 100nF, Capacitor_SMD:C_0805_2012Metric_Pad1.15x1.40mm_HandSolder, B.Cu at (167.0, 48.1)
- added C406: 100nF, Capacitor_SMD:C_0805_2012Metric_Pad1.15x1.40mm_HandSolder, B.Cu at (102.0, 48.1)
- added C501: 1uF, Capacitor_Tantalum_SMD:CP_EIA-6032-20_AVX-F_Pad2.25x2.35mm_HandSolder, B.Cu at (258.1, 95.9)
- added C501: 1uF, Capacitor_Tantalum_SMD:CP_EIA-6032-20_AVX-F_Pad2.25x2.35mm_HandSolder, B.Cu at (193.1, 95.9)
- added C501: 1uF, Capacitor_Tantalum_SMD:CP_EIA-6032-20_AVX-F_Pad2.25x2.35mm_HandSolder, B.Cu at (128.1, 95.9)
- added C502: 100nF, Capacitor_SMD:C_0805_2012Metric_Pad1.15x1.40mm_HandSolder, B.Cu at (258.1, 92.1)
- added C502: 100nF, Capacitor_SMD:C_0805_2012Metric_Pad1.15x1.40mm_HandSolder, B.Cu at (193.1, 92.1)
- added C502: 100nF, Capacitor_SMD:C_0805_2012Metric_Pad1.15x1.40mm_HandSolder, B.Cu at (128.1, 92.1)
- added C503: 100nF, Capacitor_SMD:C_0805_2012Metric_Pad1.15x1.40mm_HandSolder, B.Cu at (251.5, 95.2)
- added C503: 100nF, Capacitor_SMD:C_0805_2012Metric_Pad1.15x1.40mm_HandSolder, B.Cu at (186.5, 95.2)
- added C503: 100nF, Capacitor_SMD:C_0805_2012Metric_Pad1.15x1.40mm_HandSolder, B.Cu at (121.5, 95.2)
- added C504: 1uF, Capacitor_Tantalum_SMD:CP_EIA-6032-20_AVX-F_Pad2.25x2.35mm_HandSolder, B.Cu at (251.5, 92.1)
- added C504: 1uF, Capacitor_Tantalum_SMD:CP_EIA-6032-20_AVX-F_Pad2.25x2.35mm_HandSolder, B.Cu at (186.5, 92.1)
- added C504: 1uF, Capacitor_Tantalum_SMD:CP_EIA-6032-20_AVX-F_Pad2.25x2.35mm_HandSolder, B.Cu at (121.5, 92.1)
- added D201: pesd1can, Package_TO_SOT_SMD:SOT-23_Handsoldering, B.Cu at (246.1, 124.8)
- added D201: pesd1can, Package_TO_SOT_SMD:SOT-23_Handsoldering, B.Cu at (181.1, 124.8)
- added D201: pesd1can, Package_TO_SOT_SMD:SOT-23_Handsoldering, B.Cu at (116.1, 124.8)
- added D401: LL4148, Diode_SMD:D_MiniMELF_Handsoldering, B.Cu at (225.0, 48.3)
- added D401: LL4148, Diode_SMD:D_MiniMELF_Handsoldering, B.Cu at (160.0, 48.3)
- added D401: LL4148, Diode_SMD:D_MiniMELF_Handsoldering, B.Cu at (95.0, 48.3)
- added D402: LED_RED, LED_SMD:LED_0805_2012Metric_Pad1.15x1.40mm_HandSolder, B.Cu at (224.5, 88.4)
- added D402: LED_RED, LED_SMD:LED_0805_2012Metric_Pad1.15x1.40mm_HandSolder, B.Cu at (159.5, 88.4)
- added D402: LED_RED, LED_SMD:LED_0805_2012Metric_Pad1.15x1.40mm_HandSolder, B.Cu at (94.5, 88.4)
- added D403: LED_RED, LED_SMD:LED_0805_2012Metric_Pad1.15x1.40mm_HandSolder, B.Cu at (224.5, 85.8)
- added D403: LED_RED, LED_SMD:LED_0805_2012Metric_Pad1.15x1.40mm_HandSolder, B.Cu at (159.5, 85.8)
- added D403: LED_RED, LED_SMD:LED_0805_2012Metric_Pad1.15x1.40mm_HandSolder, B.Cu at (94.5, 85.8)
- added D501: LL4148, Diode_SMD:D_MiniMELF_Handsoldering, B.Cu at (263.6, 109.2)
- added D501: LL4148, Diode_SMD:D_MiniMELF_Handsoldering, B.Cu at (198.6, 109.2)
- added D501: LL4148, Diode_SMD:D_MiniMELF_Handsoldering, B.Cu at (133.6, 109.2)
- added F501: 500mA, Fuse:Fuse_1206_3216Metric_Pad1.42x1.75mm_HandSolder, B.Cu at (263.6, 100.3)
- added F501: 500mA, Fuse:Fuse_1206_3216Metric_Pad1.42x1.75mm_HandSolder, B.Cu at (198.6, 100.3)
- added F501: 500mA, Fuse:Fuse_1206_3216Metric_Pad1.42x1.75mm_HandSolder, B.Cu at (133.6, 100.3)
- added H101: MountingHole, MountingHole:MountingHole_3.2mm_M3, F.Cu at (222.9, 38.1)
- added H101: MountingHole, MountingHole:MountingHole_3.2mm_M3, F.Cu at (157.9, 38.1)
- added H101: MountingHole, MountingHole:MountingHole_3.2mm_M3, F.Cu at (92.9, 38.1)
- added H102: MountingHole, MountingHole:MountingHole_3.2mm_M3, F.Cu at (221.9, 122.9)
- added H102: MountingHole, MountingHole:MountingHole_3.2mm_M3, F.Cu at (156.9, 122.9)
- added H102: MountingHole, MountingHole:MountingHole_3.2mm_M3, F.Cu at (91.9, 122.9)
- added H103: MountingHole, MountingHole:MountingHole_3.2mm_M3, F.Cu at (265.1, 122.9)
- added H103: MountingHole, MountingHole:MountingHole_3.2mm_M3, F.Cu at (200.1, 122.9)
- added H103: MountingHole, MountingHole:MountingHole_3.2mm_M3, F.Cu at (135.1, 122.9)
- added H104: MountingHole, MountingHole:MountingHole_3.2mm_M3, F.Cu at (264.9, 38.1)
- added H104: MountingHole, MountingHole:MountingHole_3.2mm_M3, F.Cu at (199.8, 38.1)
- added H104: MountingHole, MountingHole:MountingHole_3.2mm_M3, F.Cu at (134.8, 38.1)
- added J1: Conn_01x04, Connector_PinHeader_2.54mm:PinHeader_1x04_P2.54mm_Vertical, F.Cu at (244.5, 38.1)
- added J1: Conn_01x04, Connector_PinHeader_2.54mm:PinHeader_1x04_P2.54mm_Vertical, F.Cu at (179.5, 38.1)
- added J1: Conn_01x04, Connector_PinHeader_2.54mm:PinHeader_1x04_P2.54mm_Vertical, F.Cu at (114.5, 38.1)
- added J1: Conn_01x04, Connector_PinHeader_2.54mm:PinHeader_1x04_P2.54mm_Vertical, F.Cu at (49.5, 38.1)
- added J401: USART, Connector_PinHeader_2.54mm:PinHeader_1x04_P2.54mm_Vertical, F.Cu at (221.9, 60.7)
- added J401: USART, Connector_PinHeader_2.54mm:PinHeader_1x04_P2.54mm_Vertical, F.Cu at (156.9, 60.7)
- added J401: USART, Connector_PinHeader_2.54mm:PinHeader_1x04_P2.54mm_Vertical, F.Cu at (91.9, 60.7)
- added J601: RJ45, KicadZeniteSolarLibrary18:RJ45_YH59_01, F.Cu at (248.6, 135.6)
- added J601: RJ45, KicadZeniteSolarLibrary18:RJ45_YH59_01, F.Cu at (183.6, 135.6)
- added J601: RJ45, KicadZeniteSolarLibrary18:RJ45_YH59_01, F.Cu at (118.6, 135.6)
- added J602: RJ45, KicadZeniteSolarLibrary18:RJ45_YH59_01, F.Cu at (227.7, 135.6)
- added J602: RJ45, KicadZeniteSolarLibrary18:RJ45_YH59_01, F.Cu at (162.7, 135.6)
- added J602: RJ45, KicadZeniteSolarLibrary18:RJ45_YH59_01, F.Cu at (97.7, 135.6)
- added R201: 120, Resistor_SMD:R_0805_2012Metric_Pad1.15x1.40mm_HandSolder, B.Cu at (246.1, 120.8)
- added R201: 120, Resistor_SMD:R_0805_2012Metric_Pad1.15x1.40mm_HandSolder, B.Cu at (181.1, 120.8)
- added R201: 120, Resistor_SMD:R_0805_2012Metric_Pad1.15x1.40mm_HandSolder, B.Cu at (116.1, 120.8)
- added R202: 4k7, Resistor_SMD:R_0805_2012Metric_Pad1.15x1.40mm_HandSolder, B.Cu at (237.8, 121.9)
- added R202: 4k7, Resistor_SMD:R_0805_2012Metric_Pad1.15x1.40mm_HandSolder, B.Cu at (172.8, 121.9)
- added R202: 4k7, Resistor_SMD:R_0805_2012Metric_Pad1.15x1.40mm_HandSolder, B.Cu at (107.8, 121.9)
- added R203: 10k, Resistor_SMD:R_0805_2012Metric_Pad1.15x1.40mm_HandSolder, B.Cu at (246.0, 108.0)
- added R203: 10k, Resistor_SMD:R_0805_2012Metric_Pad1.15x1.40mm_HandSolder, B.Cu at (181.0, 108.0)
- added R203: 10k, Resistor_SMD:R_0805_2012Metric_Pad1.15x1.40mm_HandSolder, B.Cu at (116.0, 108.0)
- added R401: 10k, Resistor_SMD:R_0805_2012Metric_Pad1.15x1.40mm_HandSolder, B.Cu at (229.5, 50.5)
- added R401: 10k, Resistor_SMD:R_0805_2012Metric_Pad1.15x1.40mm_HandSolder, B.Cu at (164.5, 50.5)
- added R401: 10k, Resistor_SMD:R_0805_2012Metric_Pad1.15x1.40mm_HandSolder, B.Cu at (99.5, 50.5)
- added R402: 1k, Resistor_SMD:R_0805_2012Metric_Pad1.15x1.40mm_HandSolder, B.Cu at (229.5, 55.6)
- added R402: 1k, Resistor_SMD:R_0805_2012Metric_Pad1.15x1.40mm_HandSolder, B.Cu at (164.5, 55.6)
- added R402: 1k, Resistor_SMD:R_0805_2012Metric_Pad1.15x1.40mm_HandSolder, B.Cu at (99.5, 55.6)
- added R403: 1k, Resistor_SMD:R_0805_2012Metric_Pad1.15x1.40mm_HandSolder, B.Cu at (229.5, 58.2)
- added R403: 1k, Resistor_SMD:R_0805_2012Metric_Pad1.15x1.40mm_HandSolder, B.Cu at (164.5, 58.2)
- added R403: 1k, Resistor_SMD:R_0805_2012Metric_Pad1.15x1.40mm_HandSolder, B.Cu at (99.5, 58.2)
- added R404: 1k, Resistor_SMD:R_0805_2012Metric_Pad1.15x1.40mm_HandSolder, B.Cu at (228.3, 88.4)
- added R404: 1k, Resistor_SMD:R_0805_2012Metric_Pad1.15x1.40mm_HandSolder, B.Cu at (163.3, 88.4)
- added R404: 1k, Resistor_SMD:R_0805_2012Metric_Pad1.15x1.40mm_HandSolder, B.Cu at (98.3, 88.4)
- added R405: 1k, Resistor_SMD:R_0805_2012Metric_Pad1.15x1.40mm_HandSolder, B.Cu at (228.3, 85.8)
- added R405: 1k, Resistor_SMD:R_0805_2012Metric_Pad1.15x1.40mm_HandSolder, B.Cu at (163.3, 85.8)
- added R405: 1k, Resistor_SMD:R_0805_2012Metric_Pad1.15x1.40mm_HandSolder, B.Cu at (98.3, 85.8)
- added TP201: SI, TestPoint:TestPoint_Pad_2.0x2.0mm, B.Cu at (250.0, 101.6)
- added TP201: SI, TestPoint:TestPoint_Pad_2.0x2.0mm, B.Cu at (185.0, 101.6)
- added TP201: SI, TestPoint:TestPoint_Pad_2.0x2.0mm, B.Cu at (120.0, 101.6)
- added TP202: SO, TestPoint:TestPoint_Pad_2.0x2.0mm, B.Cu at (250.0, 104.8)
- added TP202: SO, TestPoint:TestPoint_Pad_2.0x2.0mm, B.Cu at (185.0, 104.8)
- added TP202: SO, TestPoint:TestPoint_Pad_2.0x2.0mm, B.Cu at (120.0, 104.8)
- added TP203: TXCAN, TestPoint:TestPoint_Pad_2.0x2.0mm, B.Cu at (228.9, 112.1)
- added TP203: TXCAN, TestPoint:TestPoint_Pad_2.0x2.0mm, B.Cu at (163.9, 112.1)
- added TP203: TXCAN, TestPoint:TestPoint_Pad_2.0x2.0mm, B.Cu at (98.9, 112.1)
- added TP204: RXCAN, TestPoint:TestPoint_Pad_2.0x2.0mm, B.Cu at (228.9, 108.3)
- added TP204: RXCAN, TestPoint:TestPoint_Pad_2.0x2.0mm, B.Cu at (163.9, 108.3)
- added TP204: RXCAN, TestPoint:TestPoint_Pad_2.0x2.0mm, B.Cu at (98.9, 108.3)
- added TP205: SC, TestPoint:TestPoint_Pad_2.0x2.0mm, B.Cu at (250.0, 108.0)
- added TP205: SC, TestPoint:TestPoint_Pad_2.0x2.0mm, B.Cu at (185.0, 108.0)
- added TP205: SC, TestPoint:TestPoint_Pad_2.0x2.0mm, B.Cu at (120.0, 108.0)
- added TP206: SCK, TestPoint:TestPoint_Pad_2.0x2.0mm, B.Cu at (250.0, 98.4)
- added TP206: SCK, TestPoint:TestPoint_Pad_2.0x2.0mm, B.Cu at (185.0, 98.4)
- added TP206: SCK, TestPoint:TestPoint_Pad_2.0x2.0mm, B.Cu at (120.0, 98.4)
- added TP207: CAN_H, TestPoint:TestPoint_Pad_2.0x2.0mm, B.Cu at (244.1, 118.1)
- added TP207: CAN_H, TestPoint:TestPoint_Pad_2.0x2.0mm, B.Cu at (179.1, 118.1)
- added TP207: CAN_H, TestPoint:TestPoint_Pad_2.0x2.0mm, B.Cu at (114.1, 118.1)
- added TP208: CAN_L, TestPoint:TestPoint_Pad_2.0x2.0mm, B.Cu at (246.7, 114.7)
- added TP208: CAN_L, TestPoint:TestPoint_Pad_2.0x2.0mm, B.Cu at (181.7, 114.7)
- added TP208: CAN_L, TestPoint:TestPoint_Pad_2.0x2.0mm, B.Cu at (116.7, 114.7)
- added TP209: INT, TestPoint:TestPoint_Pad_2.0x2.0mm, B.Cu at (243.3, 89.2)
- added TP209: INT, TestPoint:TestPoint_Pad_2.0x2.0mm, B.Cu at (178.3, 89.2)
- added TP209: INT, TestPoint:TestPoint_Pad_2.0x2.0mm, B.Cu at (113.3, 89.2)
- added U201: MCP2551-I/SN, Package_SO:SOIC-8_3.9x4.9mm_P1.27mm, B.Cu at (237.8, 114.7)
- added U201: MCP2551-I/SN, Package_SO:SOIC-8_3.9x4.9mm_P1.27mm, B.Cu at (172.8, 114.7)
- added U201: MCP2551-I/SN, Package_SO:SOIC-8_3.9x4.9mm_P1.27mm, B.Cu at (107.8, 114.7)
- added U202: MCP2515-xSO, Package_SO:SOIC-18W_7.5x11.6mm_P1.27mm, B.Cu at (237.8, 102.6)
- added U202: MCP2515-xSO, Package_SO:SOIC-18W_7.5x11.6mm_P1.27mm, B.Cu at (172.8, 102.6)
- added U202: MCP2515-xSO, Package_SO:SOIC-18W_7.5x11.6mm_P1.27mm, B.Cu at (107.8, 102.6)
- added U401: ATMEGA328P-PU, Package_DIP:DIP-28_W7.62mm_Socket, F.Cu at (234.6, 53.1)
- added U401: ATMEGA328P-PU, Package_DIP:DIP-28_W7.62mm_Socket, F.Cu at (169.6, 53.1)
- added U401: ATMEGA328P-PU, Package_DIP:DIP-28_W7.62mm_Socket, F.Cu at (104.6, 53.1)
- added U501: LM7805, KicadZeniteSolarLibrary18:TO-220-3_Horizontal_TabDown_SMD, B.Cu at (257.2, 86.4)
- added U501: LM7805, KicadZeniteSolarLibrary18:TO-220-3_Horizontal_TabDown_SMD, B.Cu at (192.2, 86.4)
- added U501: LM7805, KicadZeniteSolarLibrary18:TO-220-3_Horizontal_TabDown_SMD, B.Cu at (127.2, 86.4)
- added Y201: 16MHz, Crystal:Crystal_HC49-U_Vertical, F.Cu at (227.0, 102.6)
- added Y201: 16MHz, Crystal:Crystal_HC49-U_Vertical, F.Cu at (162.0, 102.6)
- added Y201: 16MHz, Crystal:Crystal_HC49-U_Vertical, F.Cu at (97.0, 102.6)
- added Y401: 16MHz, Crystal:Crystal_HC49-U_Vertical, F.Cu at (228.3, 78.5)
- added Y401: 16MHz, Crystal:Crystal_HC49-U_Vertical, F.Cu at (163.3, 78.5)
- added Y401: 16MHz, Crystal:Crystal_HC49-U_Vertical, F.Cu at (98.3, 78.5)
- moved J602 161.4 mm to (32.7, 135.6), turned to 0 degrees
- moved H102 153.2 mm to (26.9, 122.9), turned to 270 degrees
- moved J601 145.3 mm to (53.6, 135.6), turned to 0 degrees
- moved R202 137.4 mm to (42.8, 121.9), turned to 180 degrees
- moved TP203 135.4 mm to (33.9, 112.1), turned to 270 degrees
- moved C205 135.0 mm to (42.8, 119.8), turned to 180 degrees
- moved D201 134.0 mm to (51.1, 124.8), turned to 270 degrees
- moved TP204 131.7 mm to (33.9, 108.3), turned to 270 degrees
- moved U201 129.4 mm to (42.8, 114.7), turned to 0 degrees
- moved R201 129.3 mm to (51.1, 120.8), turned to 180 degrees
- moved Y201 128.4 mm to (32.0, 102.6), turned to 90 degrees
- moved TP207 127.7 mm to (49.1, 118.1), turned to 270 degrees
- moved C203 125.7 mm to (32.4, 100.1), turned to 180 degrees
- moved TP208 121.6 mm to (51.7, 114.7), turned to 270 degrees
- moved C204 120.0 mm to (34.5, 96.3), turned to 0 degrees
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Connections:
- C102 pad 1: Net-(C102-Pad1) -> +5V
- U401 pad 23: /MCU/analog1 -> Net-(U401-Pad23)
- U401 pad 27: Net-(U401-Pad27) -> /MCU/SDA
- U401 pad 28: Net-(U401-Pad28) -> /MCU/SCL
- U501 pad : (no net) -> GND
Routing:
- net +5V: track 215.0 -> 807.1 mm
- net GND: track 99.9 -> 318.1 mm, vias 18 -> 56
- net /POWER SUPPLY/+18V_IN: track 71.9 -> 287.8 mm
- net /CANBUS CONN/CAN_H: track 50.6 -> 202.3 mm
- net /CANBUS CONN/CAN_L: track 48.2 -> 192.7 mm, vias 2 -> 8
- net /MISO: track 37.7 -> 150.9 mm
- net /SCK: track 35.6 -> 142.3 mm
- net /MOSI: track 32.9 -> 131.5 mm
- net /CANBUS/CS: track 32.2 -> 128.6 mm
- net /MCU/SDA: track 0.00 -> 92.5 mm
- net /CANBUS/INT: track 21.1 -> 84.4 mm
- net /MCU/SCL: track 0.00 -> 60.4 mm
- net /CANBUS/TXCAN: track 15.4 -> 61.4 mm
- net Net-(D101-Pad1): track 42.7 -> 0.00 mm
- net /CANBUS/RXCAN: track 14.1 -> 56.5 mm
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Other:
- board size 130.2 x 52.1 mm -> 247.1 x 121 mm
